Commit message: paddle model and URDF

File: src/pb_robot/models/franka_description/robots/hand_original.xacro (robot description, xacro)
@@ -1,5 +1,4 @@
 <?xml version="1.0" encoding="utf-8"?>
 <robot xmlns:xacro="http://www.ros.org/wiki/xacro" name="hand">
-  <xacro:include filename="$(find franka_description)/robots/paddle.xacro"/>
   <xacro:macro name="hand" params="connected_to:='' ns:='' rpy:='0 0 0' xyz:='0 0 0' ">
       <xacro:unless value="${connected_to == ''}">
@@ -63,5 +62,4 @@
         <mimic joint="${ns}_finger_joint1" />
       </joint>
-    <xacro:paddle ns="${ns}"/>
   </xacro:macro>
 </robot>

File: src/pb_robot/models/franka_description/robots/panda_arm_hand.urdf (robot description, URDF)
Before this commit: robot panda, 13 links, 12 joints
Links:
- removed link tool_link
- added link panda_paddle, mass 0.02; collision mesh filename=/home/sonam/research/pb_robot/src/pb_robot/models/franka_de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; visual mesh filename=/home/sonam/research/pb_robot/src/pb_robot/models/franka_de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
Joints:
- removed joint tool_joint
- added joint panda_paddle_joint: type fixed, parent panda_hand, child panda_paddle, origin xyz=0.0 0.0 0.1 rpy=1.57 0 0
- joint panda_hand_joint: origin xyz=0 0 0 rpy=0 0 -0.785398163397 -> xyz=0 0 0 rpy=0 0 -0.7853981633974483
- joint panda_joint2: origin xyz=0 0 0 rpy=-1.57079632679 0 0 -> xyz=0 0 0 rpy=-1.5707963267948966 0 0
- joint panda_joint3: origin xyz=0 -0.316 0 rpy=1.57079632679 0 0 -> xyz=0 -0.316 0 rpy=1.5707963267948966 0 0
- joint panda_joint4: origin xyz=0.0825 0 0 rpy=1.57079632679 0 0 -> xyz=0.0825 0 0 rpy=1.5707963267948966 0 0
- joint panda_joint5: origin xyz=-0.0825 0.384 0 rpy=-1.57079632679 0 0 -> xyz=-0.0825 0.384 0 rpy=-1.5707963267948966 0 0
- joint panda_joint6: origin xyz=0 0 0 rpy=1.57079632679 0 0 -> xyz=0 0 0 rpy=1.5707963267948966 0 0
- joint panda_joint7: origin xyz=0.088 0 0 rpy=1.57079632679 0 0 -> xyz=0.088 0 0 rpy=1.5707963267948966 0 0
